File: eagle/benchBuddy.sch (EAGLE design)
At the start: 104 parts, among them IC2 TLC274D, IC3 LM334Z, IC4 LM324D, IC5 LM324D, J1 12V_DC, J2 PHOENIX_SPRING_TERM_2POS, J4 GND, J5 3.3V, J6 5V, J7 12V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

Commit message: Added notes in schem
Other:
- note added: "1.1"
- note added: "Note: There are many parts to this schematic that were added to make the final project more useful. This includes fuses, an expansion header, and 3.3V / 5V output"
- note removed: "1.0"
Changed lines of the file:
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@@
 <text x="96.012" y="101.6" size="1.778" layer="91" rot="R90">Voltage Set</text>
 <text x="88.392" y="124.46" size="1.778" layer="91" rot="R90">Current Set</text>
-<text x="262.128" y="6.604" size="3.81" layer="94">1.0</text>
+<text x="262.128" y="6.604" size="3.81" layer="94">1.1</text>
 <text x="147.32" y="60.96" size="1.778" layer="91">Expansion Header for MCU Control</text>
 <wire x1="144.78" y1="63.5" x2="144.78" y2="0" width="0.1524" layer="97"/>
@@
 <text x="7.62" y="144.78" size="3.81" layer="97">5V @ 1A Supply</text>
 <text x="12.7" y="55.88" size="3.81" layer="97">Indicator LEDs</text>
-<text x="262.128" y="6.604" size="3.81" layer="94">1.0</text>
+<text x="262.128" y="6.604" size="3.81" layer="94">1.1</text>
+<text x="182.88" y="114.3" size="2.54" layer="97">Note: There are many parts to this schematic
+that were added to make the
+final project more useful. This includes
+fuses, an expansion header, and 3.3V / 5V output</text>
 </plain>
 <instances>

Commit message: added design rules. Gave 12V to expansion board rather than 10V. Fixed traces near 3.3V reg.
Connections:
- net 10VOLTS: no longer J3.6
- net VIN: now also J3.6
Changed lines of the file:
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@@
 <wire x1="210.82" y1="104.14" x2="210.82" y2="106.68" width="0.1524" layer="91"/>
+</segment>
+<segment>
+<pinref part="J3" gate="A" pin="6"/>
+<wire x1="152.4" y1="55.88" x2="175.26" y2="55.88" width="0.1524" layer="91"/>
+<label x="172.72" y="55.88" size="1.778" layer="95"/>
 </segment>
 </net>
@@
 <label x="264.16" y="104.14" size="1.778" layer="95"/>
 </segment>
-<segment>
-<pinref part="J3" gate="A" pin="6"/>
-<wire x1="152.4" y1="55.88" x2="175.26" y2="55.88" width="0.1524" layer="91"/>
-<label x="167.64" y="55.88" size="1.778" layer="95"/>
-</segment>
 </net>
