File: eagle/benchBuddy.brd (EAGLE design)
At the start: 114 x 76.2 mm, 104 parts, among them IC2 TLC274D, IC3 LM334Z, IC4 LM324D, IC5 LM324D, J1 12V_DC, J4 GND, J5 3.3V, J6 5V, J7 12V, J8 GND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

Commit message: Fixed acid trap issues
Routing:
- net GND: track 168.3 -> 130.0 mm, vias 16 -> 22
- net 10VOLTS: track 63.7 -> 64.7 mm
- net 3.3V: track 35.0 -> 34.3 mm

Commit message: Moved sfuse so it does not block power jack
Parts:
- moved F1 2.03 mm to (10.2, 65.5)
Routing:
- net N$3: track 6.25 -> 8.28 mm
- net N$44: track 11.7 -> 12.5 mm
Changed lines of the file:
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@@
 <?xml version="1.0" encoding="utf-8"?>
 <!DOCTYPE eagle SYSTEM "eagle.dtd">
-<eagle version="9.4.2">
+<eagle version="9.1.2">
 <drawing>
 <settings>
@@
 <attribute name="VALUE" x="40.280859375" y="23.37323125" size="0.97705625" layer="27" rot="R270"/>
 </element>
-<element name="F1" library="lab07lib" package="LITTELFUSE_MINISMDC260F/12-2" value="4A It" x="10.16" y="63.5" smashed="yes" rot="R90">
-<attribute name="NAME" x="10.707609375" y="67.048009375" size="0.98804375" layer="25" rot="R180"/>
-<attribute name="VALUE" x="13.694140625" y="60.44676875" size="0.97705625" layer="27" rot="R90"/>
+<element name="F1" library="lab07lib" package="LITTELFUSE_MINISMDC260F/12-2" value="4A It" x="10.16" y="65.532" smashed="yes" rot="R90">
+<attribute name="NAME" x="10.707609375" y="69.080009375" size="0.98804375" layer="25" rot="R180"/>
+<attribute name="VALUE" x="13.694140625" y="62.47876875" size="0.97705625" layer="27" rot="R90"/>
 </element>
 <element name="C8" library="rcl" library_urn="urn:adsk.eagle:library:334" package="C0805" package3d_urn="urn:adsk.eagle:package:23617/2" value="0.1uF" x="86.36" y="17.78" smashed="yes" rot="R90">
@@
 <contactref element="J1" pad="PWR"/>
 <wire x1="12.53" y1="55.84" x2="10.16" y2="58.21" width="2.54" layer="1"/>
-<wire x1="10.16" y1="58.21" x2="10.16" y2="61.11" width="2.54" layer="1"/>
+<wire x1="10.16" y1="58.21" x2="10.16" y2="63.142" width="2.54" layer="1"/>
 </signal>
 <signal name="N$44">
 <contactref element="F1" pad="2"/>
 <contactref element="SW4" pad="COM"/>
-<wire x1="10.16" y1="65.89" x2="15.39" y2="65.89" width="2.54" layer="1"/>
-<wire x1="15.39" y1="65.89" x2="19.05" y2="62.23" width="2.54" layer="1"/>
+<wire x1="10.16" y1="67.922" x2="13.358" y2="67.922" width="2.54" layer="1"/>
+<wire x1="13.358" y1="67.922" x2="19.05" y2="62.23" width="2.54" layer="1"/>
 <wire x1="19.05" y1="62.23" x2="19.05" y2="60.96" width="2.54" layer="1"/>
 </signal>

Commit message: Added toasty. Rotated Regs for heatsink on part sub
Parts:
- moved PS1 3.81 mm to (43.2, 10.2), turned to 0 degrees
- moved PS2 3.81 mm to (26.7, 10.2), turned to 0 degrees
Routing:
- net 5V: track 87.0 -> 79.9 mm
- net N$7: track 6.28 -> 12.9 mm
- net N$48: track 6.28 -> 12.2 mm
- net VIN: track 95.4 -> 90.0 mm
Other:
- board text added: "↓ TOASTY ↓"
Changed lines of the file:
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@@
 <setting verticaltext="up"/>
 </settings>
-<grid distance="10" unitdist="mil" unit="mil" style="lines" multiple="1" display="no" altdistance="1" altunitdist="mil" altunit="mil"/>
+<grid distance="50" unitdist="mil" unit="mil" style="lines" multiple="1" display="no" altdistance="1" altunitdist="mil" altunit="mil"/>
 <layers>
 <layer number="1" name="Top" color="4" fill="1" visible="yes" active="yes"/>
@@
 <rectangle x1="82.883709375" y1="53.914190625" x2="101.397765625" y2="53.942640625" layer="42" rot="R180"/>
 <rectangle x1="82.883709375" y1="53.942640625" x2="101.397765625" y2="53.970834375" layer="42" rot="R180"/>
+<text x="5.08" y="26.67" size="1.778" layer="21" rot="R90" align="bottom-center">↓ TOASTY ↓ </text>
 </plain>
 <attributes>
@@
 <attribute name="VENDOR" value="Texas Instruments" x="58.42" y="41.91" size="1.778" layer="27" rot="R180" display="off"/>
 </element>
-<element name="PS1" library="P78E05-1000" package="CONV_P78E05-1000" value="P78E05-1000" x="43.18" y="13.97" smashed="yes" rot="R180">
-<attribute name="MANUFACTURER" value="CUI Inc" x="43.18" y="13.97" size="1.778" layer="27" rot="R180" display="off"/>
-<attribute name="NAME" x="46.605" y="16.895" size="1.27" layer="25"/>
-<attribute name="STANDARD" value="Manufacturer Recommendations" x="43.18" y="13.97" size="1.778" layer="27" rot="R180" display="off"/>
-</element>
-<element name="PS2" library="P78E05-1000" package="CONV_P78E05-1000" value="P78E05-1000" x="26.67" y="13.97" smashed="yes" rot="R180">
-<attribute name="MANUFACTURER" value="CUI Inc" x="26.67" y="13.97" size="1.778" layer="27" rot="R180" display="off"/>
-<attribute name="NAME" x="21.205" y="17.53" size="1.27" layer="25"/>
-<attribute name="STANDARD" value="Manufacturer Recommendations" x="26.67" y="13.97" size="1.778" layer="27" rot="R180" display="off"/>
+<element name="PS1" library="P78E05-1000" package="CONV_P78E05-1000" value="P78E05-1000" x="43.18" y="10.16" smashed="yes">
+<attribute name="MANUFACTURER" value="CUI Inc" x="43.18" y="10.16" size="1.778" layer="27" display="off"/>
+<attribute name="NAME" x="45.7414" y="16.2854" size="1.27" layer="25"/>
+<attribute name="STANDARD" value="Manufacturer Recommendations" x="43.18" y="10.16" size="1.778" layer="27" display="off"/>
+</element>
+<element name="PS2" library="P78E05-1000" package="CONV_P78E05-1000" value="P78E05-1000" x="26.67" y="10.16" smashed="yes">
+<attribute name="MANUFACTURER" value="CUI Inc" x="26.67" y="10.16" size="1.778" layer="27" display="off"/>
+<attribute name="NAME" x="20.697" y="16.26" size="1.27" layer="25"/>
+<attribute name="STANDARD" value="Manufacturer Recommendations" x="26.67" y="10.16" size="1.778" layer="27" display="off"/>
 </element>
 <element name="D1" library="SparkFun-LED" library_urn="urn:adsk.eagle:library:529" package="LED_3MM" package3d_urn="urn:adsk.eagle:package:39361/1" value="" x="81.28" y="19.05" smashed="yes">
@@
 <wire x1="19.05" y1="54.61" x2="19.05" y2="52.07" width="1.27" layer="1"/>
 <wire x1="31.75" y1="23.98" x2="34.186" y2="23.98" width="1.27" layer="1"/>
-<wire x1="39.624" y1="11.684" x2="43.942" y2="11.684" width="1.27" layer="1"/>
-<wire x1="43.942" y1="11.684" x2="45.72" y2="13.462" width="1.27" layer="1"/>
-<wire x1="45.72" y1="13.462" x2="45.72" y2="13.97" width="1.27" layer="1"/>
-<wire x1="34.186" y1="23.98" x2="34.798" y2="23.368" width="1.27" layer="1"/>
-<wire x1="34.798" y1="23.368" x2="34.798" y2="16.51" width="1.27" layer="1"/>
-<wire x1="34.798" y1="16.51" x2="39.624" y2="11.684" width="1.27" layer="1"/>
+<wire x1="34.798" y1="23.368" x2="34.186" y2="23.98" width="1.27" layer="1"/>
 <contactref element="J3" pad="6"/>
+<wire x1="40.64" y1="10.16" x2="34.798" y2="16.002" width="1.27" layer="1"/>
+<wire x1="34.798" y1="16.002" x2="34.798" y2="23.368" width="1.27" layer="1"/>
+<wire x1="76.2" y1="54.67" x2="109.22" y2="63.5" width="0" layer="19" extent="1-1"/>
+<wire x1="69.774" y1="62.23" x2="76.2" y2="54.67" width="0" layer="19" extent="1-1"/>
+<wire x1="75.692" y1="41.716" x2="76.2" y2="54.67" width="0" layer="19" extent="1-1"/>
+<wire x1="61.976" y1="42.9642" x2="75.692" y2="41.716" width="0" layer="19" extent="1-16"/>
+<wire x1="80.01" y1="19.05" x2="83.312" y2="35.306" width="0" layer="19" extent="1-1"/>
+<wire x1="81.28" y1="15.24" x2="80.01" y2="19.05" width="0" layer="19" extent="1-1"/>
+<wire x1="36.89" y1="36.83" x2="55.626" y2="39.624" width="0" layer="19" extent="1-1"/>
+<wire x1="36.51" y1="29.21" x2="36.89" y2="36.83" width="0" layer="19" extent="1-1"/>
+<wire x1="34.186" y1="23.98" x2="36.51" y2="29.21" width="0" layer="19" extent="1-1"/>
+<wire x1="19.05" y1="52.07" x2="25.4" y2="42.062" width="0" layer="19" extent="1-1"/>
+<wire x1="30.48" y1="63.348" x2="23.75" y2="60.96" width="0" layer="19" extent="1-1"/>
 </signal>
 <signal name="N$1">
@@
 <wire x1="74.676" y1="16.764" x2="84.582" y2="16.764" width="0.4064" layer="16"/>
 <wire x1="72.39" y1="19.05" x2="74.676" y2="16.764" width="0.4064" layer="16"/>
-<wire x1="24.13" y1="13.97" x2="24.13" y2="12.7" width="1.27" layer="1"/>
-<wire x1="24.13" y1="12.7" x2="27.178" y2="9.652" width="1.27" layer="1"/>
-<wire x1="50.26865625" y1="9.652" x2="56.99965625" y2="2.921" width="1.27" layer="1"/>
-<wire x1="27.178" y1="9.652" x2="50.26865625" y2="9.652" width="1.27" layer="1"/>
 <wire x1="56.99965625" y1="2.921" x2="70.231" y2="2.921" width="1.27" layer="1"/>
 <wire x1="70.231" y1="2.921" x2="73.66" y2="6.35" width="1.27" layer="1"/>
+<wire x1="29.21" y1="10.16" x2="36.83" y2="2.54" width="1.27" layer="1"/>
+<wire x1="56.61865625" y1="2.54" x2="56.99965625" y2="2.921" width="1.27" layer="1"/>
+<wire x1="36.83" y1="2.54" x2="56.61865625" y2="2.54" width="1.27" layer="1"/>
 </signal>
 <signal name="3.3V">
@@
 <contactref element="PS1" pad="3"/>
 <contactref element="F2" pad="1"/>
-<wire x1="38.1" y1="19.2" x2="38.1" y2="16.51" width="1.27" layer="1"/>
-<wire x1="38.1" y1="16.51" x2="40.64" y2="13.97" width="1.27" layer="1"/>
+<wire x1="38.1" y1="19.2" x2="45.72" y2="11.58" width="1.27" layer="1"/>
+<wire x1="45.72" y1="11.58" x2="45.72" y2="10.16" width="1.27" layer="1"/>
 </signal>
 <signal name="N$49">
@@
 <contactref element="F3" pad="2"/>
 <contactref element="PS2" pad="1"/>
-<wire x1="31.75" y1="19.2" x2="31.75" y2="16.51" width="1.27" layer="1"/>
-<wire x1="31.75" y1="16.51" x2="29.21" y2="13.97" width="1.27" layer="1"/>
+<wire x1="24.13" y1="10.16" x2="24.13" y2="12.7" width="1.27" layer="1"/>
+<wire x1="24.13" y1="12.7" x2="30.63" y2="19.2" width="1.27" layer="1"/>
+<wire x1="30.63" y1="19.2" x2="31.75" y2="19.2" width="1.27" layer="1"/>
 </signal>
 </signals>

Commit message: added names
Other:
- board text added: "Mark Gilliland 2019"
- board text added: "Power Supply Bench Buddy"
Changed lines of the file:
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@@
 <rectangle x1="82.883709375" y1="53.942640625" x2="101.397765625" y2="53.970834375" layer="42" rot="R180"/>
 <text x="5.08" y="26.67" size="1.778" layer="21" rot="R90" align="bottom-center">↓ TOASTY ↓ </text>
+<text x="97.79" y="17.78" size="1.778" layer="21" align="bottom-center">Mark Gilliland
+2019</text>
+<text x="53.34" y="27.94" size="1.27" layer="21" align="bottom-center">Power Supply
+Bench Buddy</text>
 </plain>
 <attributes>
@@
 <wire x1="40.64" y1="10.16" x2="34.798" y2="16.002" width="1.27" layer="1"/>
 <wire x1="34.798" y1="16.002" x2="34.798" y2="23.368" width="1.27" layer="1"/>
-<wire x1="76.2" y1="54.67" x2="109.22" y2="63.5" width="0" layer="19" extent="1-1"/>
-<wire x1="69.774" y1="62.23" x2="76.2" y2="54.67" width="0" layer="19" extent="1-1"/>
-<wire x1="75.692" y1="41.716" x2="76.2" y2="54.67" width="0" layer="19" extent="1-1"/>
-<wire x1="61.976" y1="42.9642" x2="75.692" y2="41.716" width="0" layer="19" extent="1-16"/>
-<wire x1="80.01" y1="19.05" x2="83.312" y2="35.306" width="0" layer="19" extent="1-1"/>
-<wire x1="81.28" y1="15.24" x2="80.01" y2="19.05" width="0" layer="19" extent="1-1"/>
-<wire x1="36.89" y1="36.83" x2="55.626" y2="39.624" width="0" layer="19" extent="1-1"/>
-<wire x1="36.51" y1="29.21" x2="36.89" y2="36.83" width="0" layer="19" extent="1-1"/>
-<wire x1="34.186" y1="23.98" x2="36.51" y2="29.21" width="0" layer="19" extent="1-1"/>
-<wire x1="19.05" y1="52.07" x2="25.4" y2="42.062" width="0" layer="19" extent="1-1"/>
-<wire x1="30.48" y1="63.348" x2="23.75" y2="60.96" width="0" layer="19" extent="1-1"/>
 </signal>
 <signal name="N$1">
