File: microBackpack/microBackpack.brd (EAGLE design)
At the start: 86.4 x 76.2 mm, 96 parts, among them IC1 LM324D, IC2 LM324D, J2 USB_B, J4 2X6 FEMALE, U1 ATMEGA328P_TQFP, U10 TLP185, U11 TLP185, U2 5VREG-HS, U3 CP2102N-QFN24, U4 TVS_DIODE_4PK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

Commit message: Finished routing FGEN, added option for DIO DDS or DAC powered FGEN
Parts:
- added JP_FGEN_SEL: JUMPER-SMT_3_1-NC_PASTE_SILK, SparkFun-Jumpers:SMT-JUMPER_3_1-NC_PASTE_SILK
Connections:
- new net N$2: JP_FGEN_SEL.2, R38.2
- net DAC_C: now also JP_FGEN_SEL.3; no longer R38.2
- net DIO7_PROT: now also JP_FGEN_SEL.1
Routing:
- net DIO7_PROT: track 23.3 -> 67.8 mm, vias 0 -> 2
- net N$2: track 0.00 -> 9.28 mm
- net FGEN: track 88.9 -> 97.4 mm, vias 5 -> 1
- net DAC_C: track 9.09 -> 6.83 mm, vias 0 -> 2
- net V_SET: track 53.4 -> 54.0 mm
Changed lines of the file:
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@@
 <attribute name="VALUE" x="14.986" y="72.136" size="0.6096" layer="27" font="vector" ratio="20"/>
 </element>
+<element name="JP_FGEN_SEL" library="SparkFun-Jumpers" library_urn="urn:adsk.eagle:library:528" package="SMT-JUMPER_3_1-NC_PASTE_SILK" package3d_urn="urn:adsk.eagle:package:39293/1" value="JUMPER-SMT_3_1-NC_PASTE_SILK" x="10.922" y="39.878" smashed="yes" rot="R180"/>
 </elements>
 <signals>
@@
 <contactref element="R40" pad="1"/>
 <contactref element="U11" pad="3"/>
-<wire x1="11.7" y1="37.61" x2="11.684" y2="37.626" width="0.2032" layer="1"/>
-<wire x1="11.684" y1="37.626" x2="11.684" y2="38.862" width="0.2032" layer="1"/>
-<via x="11.684" y="38.862" extent="1-16" drill="0.254"/>
 <wire x1="31.791515625" y1="27.669828125" x2="31.0456875" y2="26.924" width="0.2032" layer="1"/>
 <wire x1="31.0456875" y1="26.924" x2="30.988" y2="26.924" width="0.2032" layer="1"/>
@@
 <wire x1="50.226" y1="62.164" x2="50.292" y2="62.23" width="0.254" layer="1"/>
 <via x="50.292" y="62.23" extent="1-16" drill="0.35"/>
+<wire x1="10.9192" y1="36.9824" x2="11.684" y2="36.9824" width="0.254" layer="1"/>
+<wire x1="10.9192" y1="36.9824" x2="10.668" y2="37.2336" width="0.254" layer="1"/>
+<via x="10.668" y="37.2336" extent="1-16" drill="0.35"/>
+<wire x1="11.684" y1="36.9824" x2="11.7" y2="36.9984" width="0.254" layer="1"/>
+<wire x1="11.7" y1="36.9984" x2="11.7" y2="37.61" width="0.254" layer="1"/>
 </signal>
 <signal name="MISO">
@@
 <wire x1="18.796" y1="40.64" x2="16.51" y2="40.64" width="0.1778" layer="16"/>
 <via x="16.51" y="40.64" extent="1-16" drill="0.35"/>
-<wire x1="16.51" y1="40.64" x2="8.128" y2="40.64" width="0.1778" layer="1"/>
+<wire x1="16.51" y1="40.64" x2="14.478" y2="40.64" width="0.1778" layer="1"/>
+<wire x1="14.478" y1="40.64" x2="13.716" y2="41.402" width="0.1778" layer="1"/>
+<wire x1="13.716" y1="41.402" x2="8.89" y2="41.402" width="0.1778" layer="1"/>
 <wire x1="6.29" y1="31.436" x2="6.29" y2="30.734" width="0.1778" layer="1"/>
-<wire x1="8.128" y1="40.64" x2="7.112" y2="39.624" width="0.1778" layer="1"/>
+<wire x1="8.89" y1="41.402" x2="7.112" y2="39.624" width="0.1778" layer="1"/>
 <wire x1="6.29" y1="31.436" x2="7.112" y2="32.258" width="0.1778" layer="1"/>
 <wire x1="30.48" y1="60.96" x2="23.876" y2="60.96" width="0.1778" layer="1"/>
@@
 <signal name="DAC_C">
 <contactref element="U5" pad="8"/>
-<contactref element="R38" pad="2"/>
-<wire x1="12.7" y1="37.61" x2="12.6294" y2="37.5394" width="0.2032" layer="1"/>
-<wire x1="12.6294" y1="37.5394" x2="12.6294" y2="36.99426875" width="0.2032" layer="1"/>
-<wire x1="12.6294" y1="36.99426875" x2="12.21113125" y2="36.576" width="0.2032" layer="1"/>
-<wire x1="12.21113125" y1="36.576" x2="9.906" y2="36.576" width="0.2032" layer="1"/>
-<wire x1="9.906" y1="36.576" x2="6.924" y2="33.594" width="0.2032" layer="1"/>
-<wire x1="6.924" y1="33.594" x2="5.588" y2="33.594" width="0.2032" layer="1"/>
+<contactref element="JP_FGEN_SEL" pad="3"/>
+<wire x1="10.1092" y1="39.878" x2="9.398" y2="39.878" width="0.254" layer="1"/>
+<wire x1="9.398" y1="39.878" x2="8.89" y2="40.386" width="0.254" layer="1"/>
+<via x="8.89" y="40.386" extent="1-16" drill="0.35"/>
+<wire x1="8.89" y1="40.386" x2="10.61" y2="38.666" width="0.254" layer="16"/>
+<wire x1="10.61" y1="38.666" x2="11.938" y2="38.666" width="0.254" layer="16"/>
+<via x="11.938" y="38.666" extent="1-16" drill="0.35"/>
+<wire x1="11.938" y1="38.666" x2="11.996" y2="38.608" width="0.254" layer="1"/>
+<wire x1="11.996" y1="38.608" x2="12.446" y2="38.608" width="0.254" layer="1"/>
+<wire x1="12.446" y1="38.608" x2="12.7" y2="38.354" width="0.254" layer="1"/>
+<wire x1="12.7" y1="38.354" x2="12.7" y2="37.61" width="0.254" layer="1"/>
 </signal>
 <signal name="DAC_D">
@@
 <wire x1="3.302" y1="41.722" x2="3.302" y2="39.558" width="0.1778" layer="1"/>
 <via x="8.89" y="42.672" extent="1-16" drill="0.35"/>
-<wire x1="8.89" y1="42.672" x2="12.954" y2="42.672" width="0.4064" layer="16"/>
-<wire x1="12.954" y1="42.672" x2="16.002" y2="39.624" width="0.4064" layer="16"/>
-<via x="24.638" y="38.862" extent="1-16" drill="0.35"/>
-<wire x1="23.876" y1="39.624" x2="24.638" y2="38.862" width="0.4064" layer="16"/>
-<wire x1="23.876" y1="39.624" x2="16.002" y2="39.624" width="0.4064" layer="16"/>
-<wire x1="24.638" y1="38.862" x2="25.908" y2="37.592" width="0.254" layer="1"/>
-<wire x1="25.908" y1="37.592" x2="25.908" y2="34.29" width="0.254" layer="1"/>
-<via x="25.908" y="34.29" extent="1-16" drill="0.35"/>
-<wire x1="25.908" y1="34.29" x2="26.416" y2="33.782" width="0.254" layer="16"/>
-<wire x1="26.416" y1="33.782" x2="26.416" y2="30.226" width="0.254" layer="16"/>
-<via x="26.416" y="30.226" extent="1-16" drill="0.35"/>
-<wire x1="46.99" y1="6.35" x2="46.99" y2="9.398" width="0.254" layer="16"/>
-<wire x1="46.99" y1="9.398" x2="46.482" y2="9.906" width="0.254" layer="16"/>
-<via x="22.86" y="23.622" extent="1-16" drill="0.35"/>
-<wire x1="26.416" y1="23.622" x2="22.86" y2="23.622" width="0.254" layer="1"/>
-<wire x1="46.482" y1="9.906" x2="39.878" y2="9.906" width="0.254" layer="16"/>
-<wire x1="39.878" y1="9.906" x2="37.084" y2="7.112" width="0.254" layer="16"/>
-<wire x1="37.084" y1="7.112" x2="35.052" y2="7.112" width="0.254" layer="16"/>
-<wire x1="35.052" y1="7.112" x2="33.274" y2="8.89" width="0.254" layer="16"/>
-<wire x1="33.274" y1="8.89" x2="26.162" y2="8.89" width="0.254" layer="16"/>
-<wire x1="26.162" y1="8.89" x2="22.86" y2="12.192" width="0.254" layer="16"/>
-<wire x1="22.86" y1="12.192" x2="22.86" y2="23.622" width="0.254" layer="16"/>
-<wire x1="26.416" y1="30.226" x2="26.416" y2="23.622" width="0.254" layer="1"/>
+<wire x1="46.99" y1="6.35" x2="46.99" y2="3.302" width="0.4064" layer="1"/>
+<wire x1="2.22" y1="39.558" x2="3.302" y2="39.558" width="0.4064" layer="1"/>
+<wire x1="46.99" y1="3.302" x2="44.704" y2="1.016" width="0.4064" layer="1"/>
+<wire x1="44.704" y1="1.016" x2="4.318" y2="1.016" width="0.4064" layer="1"/>
+<wire x1="4.318" y1="1.016" x2="1.778" y2="3.556" width="0.4064" layer="1"/>
+<wire x1="1.778" y1="3.556" x2="1.778" y2="39.116" width="0.4064" layer="1"/>
+<wire x1="1.778" y1="39.116" x2="2.22" y2="39.558" width="0.4064" layer="1"/>
 </signal>
 <signal name="N$11">
@@
 <wire x1="39.878" y1="20.066" x2="40.132" y2="20.32" width="0.254" layer="16"/>
 <via x="40.132" y="20.32" extent="1-16" drill="0.35"/>
-<wire x1="40.132" y1="20.32" x2="40.64" y2="20.32" width="0.254" layer="1"/>
-<wire x1="40.64" y1="20.32" x2="42.164" y2="18.796" width="0.254" layer="1"/>
+<wire x1="40.132" y1="20.32" x2="41.402" y2="20.32" width="0.254" layer="1"/>
+<wire x1="42.164" y1="19.558" x2="42.164" y2="18.796" width="0.254" layer="1"/>
+<wire x1="41.402" y1="20.32" x2="42.164" y2="19.558" width="0.254" layer="1"/>
 </signal>
 <signal name="DIO5_PROT">
@@
 <wire x1="41.976" y1="16.444" x2="41.976" y2="15.564" width="0.254" layer="1"/>
 <wire x1="41.3258" y1="17.0942" x2="41.976" y2="16.444" width="0.254" layer="1"/>
+<contactref element="JP_FGEN_SEL" pad="1"/>
+<wire x1="40.593775" y1="18.8948" x2="40.7388" y2="18.8948" width="0.254" layer="1"/>
+<wire x1="40.7388" y1="18.8948" x2="41.148" y2="19.304" width="0.254" layer="1"/>
+<via x="41.148" y="19.304" extent="1-16" drill="0.35"/>
+<wire x1="41.148" y1="19.304" x2="40.894" y2="19.05" width="0.254" layer="16"/>
+<wire x1="36.576" y1="19.05" x2="35.052" y2="20.574" width="0.254" layer="16"/>
+<wire x1="35.052" y1="20.574" x2="34.29" y2="20.574" width="0.254" layer="16"/>
+<wire x1="34.29" y1="20.574" x2="33.02" y2="19.304" width="0.254" layer="16"/>
+<wire x1="33.02" y1="19.304" x2="30.988" y2="19.304" width="0.254" layer="16"/>
+<wire x1="28.956" y1="21.336" x2="25.4" y2="21.336" width="0.254" layer="16"/>
+<wire x1="25.4" y1="21.336" x2="15.494" y2="31.242" width="0.254" layer="16"/>
+<wire x1="15.494" y1="31.242" x2="15.494" y2="35.814" width="0.254" layer="16"/>
+<via x="15.494" y="35.814" extent="1-16" drill="0.35"/>
+<wire x1="15.494" y1="35.814" x2="15.494" y2="39.116" width="0.254" layer="1"/>
+<wire x1="15.494" y1="39.116" x2="14.732" y2="39.878" width="0.254" layer="1"/>
+<wire x1="14.732" y1="39.878" x2="11.7348" y2="39.878" width="0.254" layer="1"/>
+<wire x1="40.894" y1="19.05" x2="36.576" y2="19.05" width="0.254" layer="16"/>
+<wire x1="30.988" y1="19.304" x2="28.956" y2="21.336" width="0.254" layer="16"/>
 </signal>
 <signal name="N$4">
@@
 <wire x1="60.706" y1="47.686" x2="62.738" y2="47.686" width="0.254" layer="1"/>
 </signal>
+<signal name="N$2">
+<contactref element="JP_FGEN_SEL" pad="2"/>
+<contactref element="R38" pad="2"/>
+<wire x1="10.922" y1="39.878" x2="10.922" y2="38.608" width="0.254" layer="1"/>
+<wire x1="7.62" y1="35.306" x2="7.62" y2="34.29" width="0.254" layer="1"/>
+<wire x1="7.62" y1="34.29" x2="6.924" y2="33.594" width="0.254" layer="1"/>
+<wire x1="6.924" y1="33.594" x2="5.588" y2="33.594" width="0.254" layer="1"/>
+<wire x1="10.922" y1="38.608" x2="7.62" y2="35.306" width="0.254" layer="1"/>
+</signal>
 </signals>
